File: RNS.brd (EAGLE design)
At the start: 75.9 x 59.7 mm, 12 parts

Commit message: Add files via upload
Parts:
- moved POWER_JACK 2.84 mm to (8.89, 36.8), turned to 270 degrees
Routing:
- net GND: track 124.1 -> 141.1 mm
- net IN: track 9.65 -> 23.5 mm

Commit message: Add files via upload
Parts:
- TTL: value USB-TTL-RED_ROV -> (none); device MIA_LIBRARY-2-2-2:USB-SERIAL-FT232R -> MIA_LIBRARY-2-2-2:1X04
- moved TTL 11.4 mm to (38.1, 17.8), turned to 0 degrees
- moved RESISTOR 8.03 mm to (35.6, 10.2), turned to 180 degrees
Connections:
- net 5V: now also TTL.3; no longer TTL.4
- net GND: now also TTL.4; no longer TTL.5
- net PA_10: now also TTL.2; no longer TTL.3
- net PA_9: now also TTL.1; no longer TTL.2
Routing:
- net 5V: track 136.6 -> 221.9 mm
- net GND: track 141.1 -> 145.4 mm
- net CATHODE: track 7.62 -> 8.98 mm
